Commit message: removes zed and flir camera
removed zed camera due to openrave warns

File: elir_description_openrave/urdf/elir.urdf (robot description, URDF)
Before this commit: robot elir_robot, 24 links, 23 joints
Links:
- removed link flir_camera
- removed link ground_sonar
- removed link zed_center
- removed link zed_depth_camera
- removed link zed_left_camera
- removed link zed_right_camera
- link base_link: geometry visual box size=0.005 0.005 0.005
Joints:
- removed joint flir_camera_joint
- removed joint ground_sonar_base
- removed joint zed_camera_joint
- removed joint zed_depth_camera_joint
- removed joint zed_left_camera_joint
- removed joint zed_right_camera_joint

File: elir_description_openrave/urdf/elir.urdf.xacro (robot description, xacro)
@@ -12,5 +12,5 @@
     <visual name = 'base_body'>
       <geometry>
-        <box size= "0.05 0.05 0.05"/>
+        <box size= "0.005 0.005 0.005"/>
       </geometry>
       <material name="silver"/>
@@ -684,101 +684,4 @@
     </inertial>
   </link>
-  <link name="zed_left_camera">
-        <visual>
-            <origin xyz="0 0 0" rpy="0 1.57 0"/>
-            <geometry>
-                <cylinder radius="0.007" length=".031"/>
-            </geometry>
-            <material name="dark_grey">
-                <color rgba="0.1 0.1 0.1 1"/>
-            </material>
-        </visual>
-    </link>
-    <link name="zed_center">
-        <visual>
-            <origin xyz="0 0 0" rpy="0 0 0"/>
-            <geometry>
-                <mesh filename="package://elir_description_openrave/meshes/ZED.stl" />
-            </geometry>
-            <material name="light_grey">
-                <color rgba="0.8 0.8 0.8 0.8"/>
-            </material>
-        </visual>
-    </link>
-  <link name="zed_right_camera">
-        <visual>
-            <origin xyz="0 0 0" rpy="0 1.57 0"/>
-            <geometry>
-                <cylinder radius="0.007" length=".031"/>
-            </geometry>
-            <material name="dark_grey">
-                <color rgba="0.1 0.1 0.1 1"/>
-            </material>
-        </visual>
-    </link>
-    <link name="zed_depth_camera" />
-    <joint name="zed_left_camera_joint" type="fixed">
-        <parent link="zed_center"/>
-        <child link="zed_left_camera"/>
-        <origin xyz="0 0.06 0" rpy="0 0 0" />
-    </joint>
-    <joint name="zed_depth_camera_joint" type="fixed">
-        <parent link="zed_left_camera"/>
-        <child link="zed_depth_camera"/>
-        <origin xyz="0 0 0" rpy="-1.5707963267948966 0 -1.5707963267948966" />
-    </joint>
-    <joint name="zed_right_camera_joint" type="fixed">
-        <parent link="zed_center"/>
-        <child link="zed_right_camera"/>
-        <origin xyz="0 -0.06 0" rpy="0 0 0" />
-    </joint>
-    <link name="flir_camera">
-        <visual>
-            <origin xyz="0 0 0" rpy="0 ${M_PI/2} 0"/>
-            <geometry>
-                <mesh filename="package://elir_description_openrave/meshes/LeptonBreakoutBoardWithLepton3.stl" scale="0.001 0.001 0.001"/>
-            </geometry>
-            <material name="light_grey">
-                <color rgba="0.8 0.8 0.8 0.8"/>
-            </material>
-        </visual>
-    </link>
-  <joint name="zed_camera_joint" type="fixed">
-    <parent link="box_link"/>
-    <child link="zed_center"/>
-    <origin rpy="0 0 0" xyz="0.17 0.0 -0.1"/>
-  </joint>
-  <joint name="flir_camera_joint" type="fixed">
-    <parent link="box_link"/>
-    <child link="flir_camera"/>
-    <origin rpy="0 0 0" xyz="0.17 0.0 -0.05"/>
-  </joint>
-  <!-- Sonares -->
-<link name="ground_sonar" >
-		<visual>
-			<geometry>
-      <mesh filename="package://elir_description_openrave/meshes/groundsonar.dae"/>
-			</geometry>
-      <origin rpy="0 ${-M_PI/2} 0" />
-    </visual>
-    <collision>
-      <geometry>
-        <mesh filename="package://elir_description_openrave/meshes/groundsonar.dae"/>
-      </geometry>
-      <origin rpy="0 ${-M_PI/2} 0" />
-    </collision>
-    <inertial>
-      <mass value="1e-5"/>
-      <inertia ixx="1e-6" ixy="0" ixz="0" iyy="1e-6" iyz="0" izz="1e-6"/>
-    </inertial>
-	</link>
-  <gazebo reference="ground_sonar">
-    <material>Gazebo/Gold</material>
-  </gazebo>
-	<joint name="ground_sonar_base" type="fixed">
-		<parent link="box_link" />
-		<child link="ground_sonar" />
-		<origin xyz="0 0 -0.155" rpy="0 ${M_PI/2} 0" />
-	</joint>
   <!-- ROS Control-->
   <!-- Juntas -->

Commit message: removes eef_ref link

File: elir_description_openrave/urdf/elir.urdf (robot description, URDF)
Before this commit: robot elir_robot, 18 links, 17 joints
Links:
- removed link eef_ref
Joints:
- removed joint eef_ref_tracao_f
- removed joint joint_eef
- added joint eef_joint: type fixed, parent tracao_f, child eef_tracao_f, origin xyz=0.233 0.0 0.0 rpy=0 0.0 0, axis 0 1 0, limit lower=-1.0 upper=2.18 effort=1000.0 velocity=0.5

File: elir_description_openrave/urdf/elir.urdf.xacro (robot description, xacro)
@@ -337,16 +337,8 @@
   </link>
   <!-- This link represents the front traction body unit that contains front traction body, claw f1 support and claw f2 support -->
-  <link name="eef_ref"/>
-  <joint name="eef_ref_tracao_f" type="fixed">
+  <joint name="eef_joint" type="fixed">
     <parent link="tracao_f"/>
-    <child link="eef_ref"/>
+    <child link="eef_tracao_f"/>
     <origin rpy="0 0.0 0" xyz="0.233 0.0 0.0"/>
-    <limit effort="1000.0" lower="-1.0" upper="2.18" velocity="0.5"/>
-    <axis xyz="0 1 0"/>
-  </joint>
-  <joint name="joint_eef" type="fixed">
-    <parent link="eef_ref"/>
-    <child link="eef_tracao_f"/>
-    <origin rpy="0 0.0 0" xyz="0.0 0.0 0.0"/>
     <limit effort="1000.0" lower="-1.0" upper="2.18" velocity="0.5"/>
     <axis xyz="0 1 0"/>

Commit message: try to open collada files with meshlab

File: elir_description_openrave/urdf/elir.urdf (robot description, URDF)
Before this commit: robot elir_robot, 17 links, 16 joints
Links:
- link box_link: geometry collision box size=0.0367 0.0367 0.279; collision box size=0.051 0.045 0.036

File: elir_description_openrave/urdf/elir.urdf.xacro (robot description, xacro)
@@ -46,7 +46,7 @@
     <visual name = 'central_claw_base'>
       <geometry>
-        <mesh filename="package://elir_description_openrave/meshes/dxl_mx106.dae"/>
-      </geometry>
-      <material name="black"/>
+        <box size="0.051 0.045 0.036 "/>
+      </geometry>
+      <material name="silver"/>
       <origin rpy="0 0 0" xyz="0.0 0.0722 0.3554"/>
     </visual>
@@ -68,5 +68,5 @@
     <collision name ='central_claw_base'>
       <geometry>
-        <mesh filename="package://elir_description_openrave/meshes/dxl_mx106.dae"/>
+        <box size="0.051 0.045 0.036 "/>
       </geometry>
       <origin rpy="0 0 0" xyz="0.0 0.0722 0.3554"/>
